Commit message: init

File: franka_description/robots/hand.urdf.xacro (robot description, xacro)
@@ -1,5 +1,12 @@
 <?xml version="1.0" encoding="utf-8"?>
 <robot xmlns:xacro="http://www.ros.org/wiki/xacro" name="hand">
-  <xacro:include filename="hand.xacro"/>
-  <xacro:hand ns="panda"/>
+  <!-- <xacro:include filename="hand.xacro"/>
+  <xacro:hand ns="panda"/> -->
+    <!-- Initialize gripper_center properties -->
+  <xacro:arg name="gripper_center" default="false" /> <!-- Default value -->
+  <xacro:property name="gripper_center" value="$(arg gripper_center)"/> <!-- Overload with launchfile argument -->
+  <xacro:arg name="gripper_center_xyz" default="0.0 0.0 0.10" /> <!-- Default value -->
+  <xacro:property name="gripper_center_xyz" value="$(arg gripper_center_xyz)"/> <!-- Overload with launchfile argument -->
+  <!-- Create the hand urdf -->
+  <xacro:hand ns="panda" gripper_center="${gripper_center}" gripper_center_xyz="${gripper_center_xyz}"/>
 </robot>

File: franka_description/robots/hand.xacro (robot description, xacro)
@@ -2,5 +2,5 @@
 <robot xmlns:xacro="http://www.ros.org/wiki/xacro" name="hand">
   <!-- safety_distance: Minimum safety distance in [m] by which the collision volumes are expanded and which is enforced during robot motions -->
-  <xacro:macro name="hand" params="connected_to:='' ns:='' rpy:='0 0 0' xyz:='0 0 0' safety_distance:=0">
+  <xacro:macro name="hand" params="connected_to:='' ns:='' rpy:='0 0 0' xyz:='0 0 0' safety_distance:=0 gripper_center:='false' gripper_center_xyz:='0.0 0.0 0.10'">
     <xacro:unless value="${connected_to == ''}">
       <joint name="${ns}_hand_joint" type="fixed">
@@ -35,4 +35,9 @@
         </geometry>
       </visual>
+      <collision>
+        <geometry>
+          <mesh filename="package://franka_description/meshes/collision/finger.stl"/>
+        </geometry>
+      </collision>
       <!-- for simulation -->
       <inertial>
@@ -50,4 +55,9 @@
         </geometry>
       </visual>
+      <collision>
+        <geometry>
+          <mesh filename="package://franka_description/meshes/collision/finger.stl"/>
+        </geometry>
+      </collision>
       <!-- for simulation -->
       <inertial>
@@ -63,5 +73,5 @@
       <origin xyz="0 0 0.0584" rpy="0 0 0"/>
       <axis xyz="0 1 0"/>
-      <limit effort="20" lower="0.0" upper="0.04" velocity="0.2"/>
+      <limit effort="1" lower="0.0" upper="0.04" velocity="0.1"/>
     </joint>
     <joint name="${ns}_finger_joint2" type="prismatic">
@@ -70,7 +80,18 @@
       <origin xyz="0 0 0.0584" rpy="0 0 0"/>
       <axis xyz="0 -1 0"/>
-      <limit effort="20" lower="0.0" upper="0.04" velocity="0.2"/>
-      <mimic joint="${ns}_finger_joint1" />
+      <limit effort="1" lower="0.0" upper="0.04" velocity="0.1"/>
+      <!-- mimic joint="${ns}_finger_joint1" /-->
     </joint>
+     <!-- Create gripper center virtual link and joint -->
+    <xacro:if value="${gripper_center}"> <!-- Only when gripper_center==True -->
+      <link name="${ns}_gripper_center">
+      </link>
+      <joint name="${ns}_gripper_center_joint" type="fixed">
+        <parent link="${ns}_hand"/>
+        <child link="${ns}_gripper_center"/>
+        <origin xyz="${gripper_center_xyz}" rpy="0 0 0"/>
+        <axis xyz="0 -1 0"/>
+      </joint>
+    </xacro:if>
   </xacro:macro>
 </robot>

File: franka_description/robots/panda_arm.urdf.xacro (robot description, xacro)
@@ -2,4 +2,9 @@
 <robot xmlns:xacro="http://www.ros.org/wiki/xacro" name="panda">
   <xacro:include filename="$(find franka_description)/robots/panda_arm.xacro" />
+  <xacro:include filename="$(find franka_description)/robots/panda.gazebo.xacro"/>
+  <xacro:include filename="panda.transmission.xacro"/>
   <xacro:panda_arm safety_distance="0.03"/>
+  <xacro:arg name="robot_name" default="panda"/>
+  <xacro:panda_gazebo robot_name="$(arg robot_name)" />
+  <xacro:panda_transmission robot_name="$(arg robot_name)" load_hand="false" />
 </robot>

File: franka_description/robots/panda_arm_hand.urdf.xacro (robot description, xacro)
@@ -1,4 +1,12 @@
 <?xml version="1.0" encoding="utf-8"?>
 <robot xmlns:xacro="http://www.ros.org/wiki/xacro" name="panda">
+  <!-- Initialize gripper_center properties -->
+  <xacro:arg name="gripper_center" default="false" />
+  <xacro:property name="gripper_center" value="$(arg gripper_center)"/>
+  <xacro:arg name="gripper_center_xyz" default="0.0 0.0 0.10" />
+  <xacro:property name="gripper_center_xyz" value="$(arg gripper_center_xyz)"/>
+  <xacro:include filename="$(find franka_description)/robots/gzplugin_grasp_fix.xacro"/>
+  <xacro:include filename="$(find franka_description)/robots/panda.transmission.xacro"/>
+  <!-- Include xacro files -->
   <xacro:include filename="$(find franka_description)/robots/panda_arm.xacro"/>
   <xacro:include filename="$(find franka_description)/robots/hand.xacro"/>
@@ -8,8 +16,9 @@
   <!-- end for simulation -->
   <xacro:panda_arm xyz="0 0 0" rpy="0 0 0" connected_to="world" arm_id="panda"/>
-  <xacro:hand ns="panda" rpy="0 0 ${-pi/4}" connected_to="panda_link8" safety_distance="0.03"/>
+  <xacro:hand ns="panda" rpy="0 0 ${-pi/4}" connected_to="panda_link8" safety_distance="0.03" gripper_center="${gripper_center}" gripper_center_xyz="${gripper_center_xyz}"/>
   <!-- for simulation -->
   <xacro:panda_gazebo arm_id="panda"/>
   <xacro:panda_control arm_id="panda" load_hand="true" />
+  <xacro:gzplugin_grasp_fix robot_name="panda"/>
   <!-- end for simulation -->
 </robot>
