Commit message: modified finger model

File: franka_description/robots/panda_arm_hand.urdf.xacro (robot description, xacro)
@@ -1,4 +1,10 @@
 <?xml version="1.0" encoding="utf-8"?>
 <robot xmlns:xacro="http://www.ros.org/wiki/xacro" name="panda">
+  <!-- <joint name="arm_mount_joint" type="fixed">
+    <parent link="mid_mount" />
+    <child link="franka_mount_link" />
+    <origin xyz="$(optenv RIDGEBACK_FRANKA_XYZ 0.21 0.0 0.0)" rpy="$(optenv RIDGEBACK_FRANKA_RPY 0 0 0)"/>
+  </joint>
+  <link name="franka_mount_link" /> -->
   <!-- Initialize gripper_center properties -->
   <xacro:arg name="gripper_center" default="false" />
@@ -17,4 +23,6 @@
   <xacro:panda_arm xyz="0 0 0" rpy="0 0 0" connected_to="world" arm_id="panda"/>
   <xacro:hand ns="panda" rpy="0 0 ${-pi/4}" connected_to="panda_link8" safety_distance="0.03" gripper_center="${gripper_center}" gripper_center_xyz="${gripper_center_xyz}"/>
+<!--   <xacro:panda_arm connected_to="franka_mount_link"/>
+ -->
   <!-- for simulation -->
   <xacro:panda_gazebo robot_name="panda"/>
